Commit message: feat: refresh robot description and sim launch

File: mtt_description/urdf/robot.urdf.xacro (robot description, xacro)
@@ -60,5 +60,5 @@
     </inertial>
     </link>
-    <joint name="1_continuous" type="continuous">
+    <joint name="1_continuous" type="fixed">
     <origin xyz="0.7014675763219452298 -0.30260966897135904707 0.29942602155526376606" rpy="1.570796326794896558 -0 -7.5633943552588769595e-16" />
     <parent link="base_link" />
@@ -98,5 +98,5 @@
     </inertial>
     </link>
-    <joint name="2_continuous" type="continuous">
+    <joint name="2_continuous" type="fixed">
     <origin xyz="0.63021293776953013488 -0.30260966897135899156 0.24925922731169392055" rpy="1.570796326794896558 -0 -7.5633943552588769595e-16" />
     <parent link="base_link" />
@@ -136,5 +136,5 @@
     </inertial>
     </link>
-    <joint name="3_continuous" type="continuous">
+    <joint name="3_continuous" type="fixed">
     <origin xyz="0.55767703136521962204 -0.30260966897135893605 0.20171053820694723191" rpy="1.570796326794896558 -0 -7.5633943552588769595e-16" />
     <parent link="base_link" />
@@ -174,5 +174,5 @@
     </inertial>
     </link>
-    <joint name="4_continuous" type="continuous">
+    <joint name="4_continuous" type="fixed">
     <origin xyz="0.47434412390430480411 -0.30260966897135888054 0.17622412429685807567" rpy="1.570796326794896558 -0 -7.5633943552588769595e-16" />
     <parent link="base_link" />
@@ -212,5 +212,5 @@
     </inertial>
     </link>
-    <joint name="5_continuous" type="continuous">
+    <joint name="5_continuous" type="fixed">
     <origin xyz="0.39101121644338021621 -0.30260966897135876952 0.15073771038676886391" rpy="1.570796326794896558 -0 -7.5633943552588769595e-16" />
     <parent link="base_link" />
@@ -250,5 +250,5 @@
     </inertial>
     </link>
-    <joint name="6_continuous" type="continuous">
+    <joint name="6_continuous" type="fixed">
     <origin xyz="0.30589785624702453548 -0.30260966897135871401 0.13716525069048957075" rpy="1.570796326794896558 -0 -7.5633943552588769595e-16" />
     <parent link="base_link" />
@@ -288,5 +288,5 @@
     </inertial>
     </link>
-    <joint name="7_continuous" type="continuous">
+    <joint name="7_continuous" type="fixed">
     <origin xyz="0.21875469438405417688 -0.3026096689713586585 0.13717527124629197433" rpy="1.570796326794896558 -0 -7.5633943552588769595e-16" />
     <parent link="base_link" />
@@ -326,5 +326,5 @@
     </inertial>
     </link>
-    <joint name="8_continuous" type="continuous">
+    <joint name="8_continuous" type="fixed">
     <origin xyz="0.13161153252108562239 -0.3026096689713586585 0.13718529180209448892" rpy="1.570796326794896558 -0 -7.5633943552588769595e-16" />
     <parent link="base_link" />
@@ -364,5 +364,5 @@
     </inertial>
     </link>
-    <joint name="9_continuous" type="continuous">
+    <joint name="9_continuous" type="fixed">
     <origin xyz="0.044468370658119274474 -0.30260966897135854747 0.13719531235789694801" rpy="1.570796326794896558 -0 -7.5633943552588769595e-16" />
     <parent link="base_link" />
@@ -402,5 +402,5 @@
     </inertial>
     </link>
-    <joint name="10_continuous" type="continuous">
+    <joint name="10_continuous" type="fixed">
     <origin xyz="-0.042674791204848093462 -0.30260966897135843645 0.13720533291369940709" rpy="1.570796326794896558 -0 -7.5633943552588769595e-16" />
     <parent link="base_link" />
@@ -440,5 +440,5 @@
     </inertial>
     </link>
-    <joint name="11_continuous" type="continuous">
+    <joint name="11_continuous" type="fixed">
     <origin xyz="-0.12981795306781560018 -0.30260966897135843645 0.13721535346950286538" rpy="1.570796326794896558 -0 -7.5633943552588769595e-16" />
     <parent link="base_link" />
@@ -478,5 +478,5 @@
     </inertial>
     </link>
-    <joint name="12_continuous" type="continuous">
+    <joint name="12_continuous" type="fixed">
     <origin xyz="-0.21696111493078301669 -0.30260966897135832543 0.13722537402530532447" rpy="1.570796326794896558 -0 -7.5633943552588769595e-16" />
     <parent link="base_link" />
@@ -516,5 +516,5 @@
     </inertial>
     </link>
-    <joint name="13_continuous" type="continuous">
+    <joint name="13_continuous" type="fixed">
     <origin xyz="-0.30410427679375034993 -0.30260966897135821441 0.13723539458110778355" rpy="1.570796326794896558 -0 -7.5633943552588769595e-16" />
     <parent link="base_link" />
@@ -554,5 +554,5 @@
     </inertial>
     </link>
-    <joint name="14_continuous" type="continuous">
+    <joint name="14_continuous" type="fixed">
     <origin xyz="-0.39124743865671768317 -0.30260966897135821441 0.13724541513691029815" rpy="1.570796326794896558 -0 -7.5633943552588769595e-16" />
     <parent link="base_link" />
@@ -592,5 +592,5 @@
     </inertial>
     </link>
-    <joint name="15_continuous" type="continuous">
+    <joint name="15_continuous" type="fixed">
     <origin xyz="-0.47839060051968412823 -0.30260966897135821441 0.13725543569271270172" rpy="1.570796326794896558 -0 -7.5633943552588769595e-16" />
     <parent link="base_link" />
@@ -630,5 +630,5 @@
     </inertial>
     </link>
-    <joint name="16_continuous" type="continuous">
+    <joint name="16_continuous" type="fixed">
     <origin xyz="-0.56553376238265151699 -0.30260966897135799236 0.13726545624851521632" rpy="1.570796326794896558 -0 -7.5633943552588769595e-16" />
     <parent link="base_link" />
@@ -668,5 +668,5 @@
     </inertial>
     </link>
-    <joint name="17_continuous" type="continuous">
+    <joint name="17_continuous" type="fixed">
     <origin xyz="-0.65267692424561885023 -0.30260966897135799236 0.13727547680431761989" rpy="1.570796326794896558 -0 -7.5633943552588769595e-16" />
     <parent link="base_link" />
@@ -706,5 +706,5 @@
     </inertial>
     </link>
-    <joint name="18_continuous" type="continuous">
+    <joint name="18_continuous" type="fixed">
     <origin xyz="-0.73982008610858640552 -0.30260966897135788134 0.13728549736012013449" rpy="1.570796326794896558 -0 -7.5633943552588769595e-16" />
     <parent link="base_link" />
@@ -744,5 +744,5 @@
     </inertial>
     </link>
-    <joint name="19_continuous" type="continuous">
+    <joint name="19_continuous" type="fixed">
     <origin xyz="-0.82595460894701899779 -0.30260966897135777032 0.14666682073043030288" rpy="1.570796326794896558 -0 -7.5633943552588769595e-16" />
     <parent link="base_link" />
@@ -782,5 +782,5 @@
     </inertial>
     </link>
-    <joint name="20_continuous" type="continuous">
+    <joint name="20_continuous" type="fixed">
     <origin xyz="-0.91110403062049183376 -0.30260966897135777032 0.16520075578373016878" rpy="1.570796326794896558 -0 -7.5633943552588769595e-16" />
     <parent link="base_link" />
@@ -1230,4 +1230,76 @@
   <origin xyz="0.62 -0.266 0.355" rpy="0 0 ${pi/2}"/>
 </joint>
+<!-- Hesai driver compatibility frame.
+     The live stack publishes point clouds with frame_id=hesai_lidar while the
+     MTT URDF uses center_lidar_link as the physical mount point. Keep both
+     names in the TF tree so mapping, Foxglove, and bags see one connected tree. -->
+<link name="hesai_lidar"/>
+<joint name="hesai_lidar_joint" type="fixed">
+  <parent link="center_lidar_link"/>
+  <child link="hesai_lidar"/>
+  <origin xyz="0 0 0" rpy="0 0 0"/>
+</joint>
+<!-- Runtime sensor mounts observed on the live robot snapshot.
+     These were previously only present in the old norlab_robot/main.urdf tree,
+     which left the current MTT description without the real sensor chain. Keep
+     them here so /robot_description matches the frames published by the live
+     stack. Field measurements should still confirm these poses later. -->
+<link name="imu_link"/>
+<joint name="imu_joint" type="fixed">
+  <parent link="hesai_lidar"/>
+  <child link="imu_link"/>
+  <origin xyz="0.0 0.0 0.061" rpy="3.141596 0 0"/>
+</joint>
+<link name="mti10_imu_link_right"/>
+<joint name="mti10_imu_joint_right" type="fixed">
+  <parent link="hesai_lidar"/>
+  <child link="mti10_imu_link_right"/>
+  <origin xyz="-0.295 -0.030 -0.785" rpy="0 1.570796 0"/>
+</joint>
+<link name="mti10_imu_link_left"/>
+<joint name="mti10_imu_joint_left" type="fixed">
+  <parent link="hesai_lidar"/>
+  <child link="mti10_imu_link_left"/>
+  <origin xyz="0.295 -0.030 -0.785" rpy="0 1.570796 3.141596"/>
+</joint>
+<link name="zed_camera_link"/>
+<joint name="zed2i_mount_joint" type="fixed">
+  <parent link="hesai_lidar"/>
+  <child link="zed_camera_link"/>
+  <origin xyz="0.0 -0.47 -0.1627" rpy="0.0 0.0 -1.57079"/>
+</joint>
+<!-- ZED 2i internal frames (matches zed_macro.urdf.xacro for model=zed2i, name=zed).
+     Normally published at runtime by the ZED SDK driver via /tf_static.
+     Defined here so the full TF tree is available during bag replay (no driver). -->
+<link name="zed_camera_center"/>
+<joint name="zed_camera_center_joint" type="fixed">
+  <parent link="zed_camera_link"/>
+  <child link="zed_camera_center"/>
+  <origin xyz="0 0 0.015" rpy="0 0 0"/>
+</joint>
+<link name="zed_left_camera_frame"/>
+<joint name="zed_left_camera_joint" type="fixed">
+  <parent link="zed_camera_center"/>
+  <child link="zed_left_camera_frame"/>
+  <origin xyz="-0.01 0.06 0" rpy="0 0 0"/>
+</joint>
+<link name="zed_left_camera_frame_optical"/>
+<joint name="zed_left_camera_joint_optical" type="fixed">
+  <parent link="zed_left_camera_frame"/>
+  <child link="zed_left_camera_frame_optical"/>
+  <origin xyz="0 0 0" rpy="-1.5707963 0.0 -1.5707963"/>
+</joint>
+<link name="zed_right_camera_frame"/>
+<joint name="zed_right_camera_joint" type="fixed">
+  <parent link="zed_camera_center"/>
+  <child link="zed_right_camera_frame"/>
+  <origin xyz="-0.01 -0.06 0" rpy="0 0 0"/>
+</joint>
+<link name="zed_right_camera_frame_optical"/>
+<joint name="zed_right_camera_joint_optical" type="fixed">
+  <parent link="zed_right_camera_frame"/>
+  <child link="zed_right_camera_frame_optical"/>
+  <origin xyz="0 0 0" rpy="-1.5707963 0.0 -1.5707963"/>
+</joint>
 <!-- Front LiDAR -->
 <link name="front_lidar_link">
@@ -1278,4 +1350,81 @@
   <origin xyz="0.01 -0.266 0.3302" rpy="0 0 0"/>
 </joint>
+<!-- RoboSense RS Bpearl runtime frame.
+     The old live robot description carried a measured rsairy mount that is not
+     the same as the generic rear_lidar_link added for simulation. Keep the
+     runtime frame here with its observed pose so the rear LiDAR and OAK tree
+     line up with the real sensor stack. -->
+<link name="rsairy"/>
+<joint name="rsairy_mount_joint" type="fixed">
+  <parent link="hesai_lidar"/>
+  <child link="rsairy"/>
+  <!-- Calibrated 2026-04-21 with calibrate_static_bag.py (P2P→P2Pl→GICP on bag_0.mcap).
+       Previous (nominal): xyz="0.125 0.86 0.0" rpy="0.0 -1.91986 -1.5707"
+       ICP result: Δt=7.74cm Δr=0.95° vs nominal. RMSE=3.07cm at voxel=2cm. -->
+  <origin xyz="0.060281 0.850474 -0.020308" rpy="3.115775 -1.215034 1.582805"/>
+</joint>
+<!-- OAK-D base mount.
+     DepthAI publishes the internal camera frames under the `oak` base frame,
+     but the live stack does not launch a dedicated oak_state_publisher node.
+     Anchor the `oak` base frame directly in the main robot description so the
+     OAK subtree joins the vehicle TF tree through robot_state_publisher. -->
+<link name="oak"/>
+<joint name="oak_mount_joint" type="fixed">
+  <parent link="rsairy"/>
+  <child link="oak"/>
+  <!-- Calibrated 2026-04-21 with calibrate_static_bag.py (camera_lidar, bag_0.mcap).
+       Previous (nominal): xyz="0.05 0.0 0.0" rpy="0.0 -1.57079 0.0"
+       Edge-based refinement: Δt=1.27cm Δr=0.171° vs nominal.
+       RPY near gimbal lock (pitch≈-π/2): representation differs but rotation is equivalent. -->
+  <origin xyz="0.049811 0.002056 -0.012516" rpy="-2.504975 -1.569137 2.507449"/>
+</joint>
+<!-- OAK-D internal frames (matches depthai_macro.urdf.xacro, name=oak, baseline=0.075, no rs_compat).
+     Normally published at runtime by the DepthAI driver via /tf_static from EEPROM calibration.
+     Positions here match the depthai_descriptions defaults; live driver overrides with device values. -->
+<link name="oak_rgb_camera_frame"/>
+<joint name="oak_rgb_camera_joint" type="fixed">
+  <parent link="oak"/>
+  <child link="oak_rgb_camera_frame"/>
+  <origin xyz="0 0 0" rpy="0 0 0"/>
+</joint>
+<link name="oak_rgb_camera_optical_frame"/>
+<joint name="oak_rgb_camera_optical_joint" type="fixed">
+  <parent link="oak_rgb_camera_frame"/>
+  <child link="oak_rgb_camera_optical_frame"/>
+  <origin xyz="0 0 0" rpy="-1.5707963 0.0 -1.5707963"/>
+</joint>
+<link name="oak_left_camera_frame"/>
+<joint name="oak_left_camera_joint" type="fixed">
+  <parent link="oak"/>
+  <child link="oak_left_camera_frame"/>
+  <origin xyz="0 0.0375 0" rpy="0 0 0"/>
+</joint>
+<link name="oak_left_camera_optical_frame"/>
+<joint name="oak_left_camera_optical_joint" type="fixed">
+  <parent link="oak_left_camera_frame"/>
+  <child link="oak_left_camera_optical_frame"/>
+  <origin xyz="0 0 0" rpy="-1.5707963 0.0 -1.5707963"/>
+</joint>
+<link name="oak_right_camera_frame"/>
+<joint name="oak_right_camera_joint" type="fixed">
+  <parent link="oak"/>
+  <child link="oak_right_camera_frame"/>
+  <origin xyz="0 -0.0375 0" rpy="0 0 0"/>
+</joint>
+<link name="oak_right_camera_optical_frame"/>
+<joint name="oak_right_camera_optical_joint" type="fixed">
+  <parent link="oak_right_camera_frame"/>
+  <child link="oak_right_camera_optical_frame"/>
+  <origin xyz="0 0 0" rpy="-1.5707963 0.0 -1.5707963"/>
+</joint>
+<!-- ZED 2i IMU frame.
+     Published at runtime by the ZED SDK from device calibration (parent: zed_left_camera_frame).
+     Position here is the nominal ZED2i value (IMU is ~26mm behind, 1mm right of left lens). -->
+<link name="zed_imu_link"/>
+<joint name="zed_imu_joint" type="fixed">
+  <parent link="zed_left_camera_frame"/>
+  <child link="zed_imu_link"/>
+  <origin xyz="-0.026 0.001 0" rpy="0 0 0"/>
+</joint>
 <!-- Legacy LiDAR (kept for compatibility) -->
 <joint name="lidar_joint" type="fixed">
@@ -1284,7 +1433,25 @@
   <origin xyz="0 0 0.8" rpy="0 0 0"/>
 </joint>
-<!-- GPS Left Antenna (Emlid Reach RS) -->
-<!-- Mounted left of the center mast, same height as lidar top + 15cm -->
-<!-- Baseline between antennas: ~1.1m — mirrors norlab_robot/urdf/main.urdf -->
+<!-- GPS Rover Antenna (Emlid Reach RS — single rover, RTK via LoRa from external base) -->
+<!-- Approximate live mount: right side, roughly midway between the Hesai and rear RS/OAK cluster. -->
+<!-- Position is intentionally approximate until the mast is re-measured on the robot. -->
+<!-- The base station is off-robot (fixed tripod); its ROS frame is not in this URDF. -->
+<link name="gps_rover_link">
+  <inertial>
+    <origin xyz="0 0 0" rpy="0 0 0"/>
+    <mass value="0.3"/>
+    <inertia ixx="0.0001" ixy="0.0" ixz="0.0" iyy="0.0001" iyz="0.0" izz="0.0001"/>
+  </inertial>
+</link>
+<joint name="gps_rover_joint" type="fixed">
+  <parent link="reference_point"/>
+  <child link="gps_rover_link"/>
+  <!-- x: approximately midway between Hesai (0.62) and rear sensor bracket (0.01) -->
+  <!-- y: ~20 cm to the robot right of the rear sensor line                         -->
+  <!-- z: mast above the rear sensor stack                                          -->
+  <origin xyz="0.315 -0.466 0.55" rpy="0 0 0"/>
+</joint>
+<!-- GPS Left Antenna (Emlid Reach RS — dual-antenna legacy, kept for reference) -->
+<!-- Only used when gps_antennas:=dual. Not active in single-rover mode.          -->
 <link name="gps_left_link">
   <inertial>
@@ -1299,5 +1466,5 @@
   <origin xyz="0.0 0.55 0.15" rpy="0 0 0"/>
 </joint>
-<!-- GPS Right Antenna (Emlid Reach RS) -->
+<!-- GPS Right Antenna (Emlid Reach RS — dual-antenna legacy) -->
 <link name="gps_right_link">
   <inertial>

File: mtt_description/urdf/robot_less_collision.urdf.xacro (robot description, xacro)
@@ -1101,4 +1101,40 @@
   <origin xyz="0.62 -0.266 0.355" rpy="0 0 ${pi/2}"/>
 </joint>
+<!-- Hesai driver compatibility frame.
+     Keep the same center LiDAR alias as the real robot so point clouds,
+     mapping, and TF consumers see one consistent tree in sim and live runs. -->
+<link name="hesai_lidar"/>
+<joint name="hesai_lidar_joint" type="fixed">
+  <parent link="center_lidar_link"/>
+  <child link="hesai_lidar"/>
+  <origin xyz="0 0 0" rpy="0 0 0"/>
+</joint>
+<!-- Runtime sensor mounts mirrored from the live robot description.
+     These frames do not drive Gazebo sensors directly, but keeping them in the
+     simulation model makes the TF tree match the real platform more closely. -->
+<link name="imu_link"/>
+<joint name="imu_joint" type="fixed">
+  <parent link="hesai_lidar"/>
+  <child link="imu_link"/>
+  <origin xyz="0.0 0.0 0.061" rpy="3.141596 0 0"/>
+</joint>
+<link name="mti10_imu_link_right"/>
+<joint name="mti10_imu_joint_right" type="fixed">
+  <parent link="hesai_lidar"/>
+  <child link="mti10_imu_link_right"/>
+  <origin xyz="-0.295 -0.030 -0.785" rpy="0 1.570796 0"/>
+</joint>
+<link name="mti10_imu_link_left"/>
+<joint name="mti10_imu_joint_left" type="fixed">
+  <parent link="hesai_lidar"/>
+  <child link="mti10_imu_link_left"/>
+  <origin xyz="0.295 -0.030 -0.785" rpy="0 1.570796 3.141596"/>
+</joint>
+<link name="zed_camera_link"/>
+<joint name="zed2i_mount_joint" type="fixed">
+  <parent link="hesai_lidar"/>
+  <child link="zed_camera_link"/>
+  <origin xyz="0.0 -0.47 -0.1627" rpy="0.0 0.0 -1.57079"/>
+</joint>
 <!-- Front LiDAR -->
 <link name="front_lidar_link">
@@ -1149,4 +1185,18 @@
   <origin xyz="0.01 -0.266 0.3302" rpy="0 0 0"/>
 </joint>
+<!-- RoboSense RS Bpearl runtime frame mirrored from the live stack. -->
+<link name="rsairy"/>
+<joint name="rsairy_mount_joint" type="fixed">
+  <parent link="hesai_lidar"/>
+  <child link="rsairy"/>
+  <origin xyz="0.060281 0.850474 -0.020308" rpy="3.115775 -1.215034 1.582805"/>
+</joint>
+<!-- OAK-D base mount mirrored from the live stack. -->
+<link name="oak"/>
+<joint name="oak_mount_joint" type="fixed">
+  <parent link="rsairy"/>
+  <child link="oak"/>
+  <origin xyz="0.049811 0.002056 -0.012516" rpy="-2.504975 -1.569137 2.507449"/>
+</joint>
 <!-- Legacy LiDAR (kept for compatibility) -->
 <joint name="lidar_joint" type="fixed">
@@ -1154,4 +1204,43 @@
   <child link="lidar_link"/>
   <origin xyz="0 0 0.8" rpy="0 0 0"/>
+</joint>
+<!-- GPS Rover Antenna (single rover setup used on the live platform). -->
+<!-- Approximate right-side midpoint mount mirrored from the live robot TF. -->
+<link name="gps_rover_link">
+  <inertial>
+    <origin xyz="0 0 0" rpy="0 0 0"/>
+    <mass value="0.3"/>
+    <inertia ixx="0.0001" ixy="0.0" ixz="0.0" iyy="0.0001" iyz="0.0" izz="0.0001"/>
+  </inertial>
+</link>
+<joint name="gps_rover_joint" type="fixed">
+  <parent link="reference_point"/>
+  <child link="gps_rover_link"/>
+  <origin xyz="0.315 -0.466 0.55" rpy="0 0 0"/>
+</joint>
+<!-- Dual-antenna legacy frames kept for compatibility with existing tools. -->
+<link name="gps_left_link">
+  <inertial>
+    <origin xyz="0 0 0" rpy="0 0 0"/>
+    <mass value="0.3"/>
+    <inertia ixx="0.0001" ixy="0.0" ixz="0.0" iyy="0.0001" iyz="0.0" izz="0.0001"/>
+  </inertial>
+</link>
+<joint name="gps_left_joint" type="fixed">
+  <parent link="center_lidar_link"/>
+  <child link="gps_left_link"/>
+  <origin xyz="0.0 0.55 0.15" rpy="0 0 0"/>
+</joint>
+<link name="gps_right_link">
+  <inertial>
+    <origin xyz="0 0 0" rpy="0 0 0"/>
+    <mass value="0.3"/>
+    <inertia ixx="0.0001" ixy="0.0" ixz="0.0" iyy="0.0001" iyz="0.0" izz="0.0001"/>
+  </inertial>
+</link>
+<joint name="gps_right_joint" type="fixed">
+  <parent link="center_lidar_link"/>
+  <child link="gps_right_link"/>
+  <origin xyz="0.0 -0.55 0.15" rpy="0 0 0"/>
 </joint>
 <!-- Gazebo sensor plugin for Center LiDAR -->

File: mtt_description/urdf/robot_no_collision.urdf.xacro (robot description, xacro)
@@ -1045,4 +1045,34 @@
   <origin xyz="0.62 -0.266 0.355" rpy="0 0 ${pi/2}"/>
 </joint>
+<link name="hesai_lidar"/>
+<joint name="hesai_lidar_joint" type="fixed">
+  <parent link="center_lidar_link"/>
+  <child link="hesai_lidar"/>
+  <origin xyz="0 0 0" rpy="0 0 0"/>
+</joint>
+<link name="imu_link"/>
+<joint name="imu_joint" type="fixed">
+  <parent link="hesai_lidar"/>
+  <child link="imu_link"/>
+  <origin xyz="0.0 0.0 0.061" rpy="3.141596 0 0"/>
+</joint>
+<link name="mti10_imu_link_right"/>
+<joint name="mti10_imu_joint_right" type="fixed">
+  <parent link="hesai_lidar"/>
+  <child link="mti10_imu_link_right"/>
+  <origin xyz="-0.295 -0.030 -0.785" rpy="0 1.570796 0"/>
+</joint>
+<link name="mti10_imu_link_left"/>
+<joint name="mti10_imu_joint_left" type="fixed">
+  <parent link="hesai_lidar"/>
+  <child link="mti10_imu_link_left"/>
+  <origin xyz="0.295 -0.030 -0.785" rpy="0 1.570796 3.141596"/>
+</joint>
+<link name="zed_camera_link"/>
+<joint name="zed2i_mount_joint" type="fixed">
+  <parent link="hesai_lidar"/>
+  <child link="zed_camera_link"/>
+  <origin xyz="0.0 -0.47 -0.1627" rpy="0.0 0.0 -1.57079"/>
+</joint>
 <!-- Front LiDAR -->
 <link name="front_lidar_link">
@@ -1092,4 +1122,16 @@
   <child link="rear_lidar_link"/>
   <origin xyz="0.01 -0.266 0.3302" rpy="0 0 0"/>
+</joint>
+<link name="rsairy"/>
+<joint name="rsairy_mount_joint" type="fixed">
+  <parent link="hesai_lidar"/>
+  <child link="rsairy"/>
+  <origin xyz="0.125 0.86 0.0" rpy="0.0 -1.91986 -1.5707"/>
+</joint>
+<link name="oak"/>
+<joint name="oak_mount_joint" type="fixed">
+  <parent link="rsairy"/>
+  <child link="oak"/>
+  <origin xyz="0.05 0.0 0.0" rpy="0.0 -1.57079 0.0"/>
 </joint>
 <!-- Legacy LiDAR (kept for compatibility) -->
