Commit message: stabilize MTT stack

File: mtt_description/urdf/robot.urdf.xacro (robot description, xacro)
@@ -1116,5 +1116,5 @@
     <child link="joint_remorque_simple" />
     <axis xyz="0 0 1"/>
-    <limit effort="1000000000.0" velocity="20" lower="-1.0471975511965976313" upper="1.0471975511965976313"/>
+    <limit effort="1000000000.0" velocity="20" lower="-0.78539816339744830962" upper="0.78539816339744830962"/>
     <physics>
     <simbody></simbody>

File: mtt_description/urdf/robot_less_collision.urdf.xacro (robot description, xacro)
@@ -982,5 +982,5 @@
     <child link="joint_remorque_simple" />
     <axis xyz="0 0 1"/>
-    <limit effort="1000000000.0" velocity="20" lower="-1.0471975511965976313" upper="1.0471975511965976313"/>
+    <limit effort="1000000000.0" velocity="20" lower="-0.78539816339744830962" upper="0.78539816339744830962"/>
     <physics>
     <simbody></simbody>
@@ -1110,5 +1110,5 @@
   <parent link="hesai_lidar"/>
   <child link="imu_link"/>
-  <origin xyz="0.0 0.0 0.061" rpy="3.141596 0 0"/>
+  <origin xyz="${imu_calib_xyz}" rpy="${imu_calib_rpy}"/>
 </joint>
 <link name="mti10_imu_link_right"/>
@@ -1116,5 +1116,5 @@
   <parent link="hesai_lidar"/>
   <child link="mti10_imu_link_right"/>
-  <origin xyz="-0.295 -0.030 -0.785" rpy="0 1.570796 0"/>
+  <origin xyz="${mti10_right_calib_xyz}" rpy="${mti10_right_calib_rpy}"/>
 </joint>
 <link name="mti10_imu_link_left"/>
@@ -1122,5 +1122,5 @@
   <parent link="hesai_lidar"/>
   <child link="mti10_imu_link_left"/>
-  <origin xyz="0.295 -0.030 -0.785" rpy="0 1.570796 3.141596"/>
+  <origin xyz="${mti10_left_calib_xyz}" rpy="${mti10_left_calib_rpy}"/>
 </joint>
 <link name="zed_camera_link"/>
@@ -1128,5 +1128,5 @@
   <parent link="hesai_lidar"/>
   <child link="zed_camera_link"/>
-  <origin xyz="0.0 -0.47 -0.1627" rpy="0.0 0.0 -1.57079"/>
+  <origin xyz="${zed2i_calib_xyz}" rpy="${zed2i_calib_rpy}"/>
 </joint>
 <!-- ZED 2i internal frames.
@@ -1217,5 +1217,5 @@
   <parent link="hesai_lidar"/>
   <child link="rsairy"/>
-  <origin xyz="0.060281 0.850474 -0.020308" rpy="3.115775 -1.215034 1.582805"/>
+  <origin xyz="${rsairy_calib_xyz}" rpy="${rsairy_calib_rpy}"/>
 </joint>
 <!-- OAK-D base mount mirrored from the live stack. -->

File: mtt_description/urdf/robot_no_collision.urdf.xacro (robot description, xacro)
@@ -926,5 +926,5 @@
     <child link="joint_remorque_simple" />
     <axis xyz="0 0 1"/>
-    <limit effort="1000000000.0" velocity="20" lower="-1.0471975511965976313" upper="1.0471975511965976313"/>
+    <limit effort="1000000000.0" velocity="20" lower="-0.78539816339744830962" upper="0.78539816339744830962"/>
     <physics>
     <simbody></simbody>
@@ -1051,5 +1051,5 @@
   <parent link="hesai_lidar"/>
   <child link="imu_link"/>
-  <origin xyz="0.0 0.0 0.061" rpy="3.141596 0 0"/>
+  <origin xyz="${imu_calib_xyz}" rpy="${imu_calib_rpy}"/>
 </joint>
 <link name="mti10_imu_link_right"/>
@@ -1057,5 +1057,5 @@
   <parent link="hesai_lidar"/>
   <child link="mti10_imu_link_right"/>
-  <origin xyz="-0.295 -0.030 -0.785" rpy="0 1.570796 0"/>
+  <origin xyz="${mti10_right_calib_xyz}" rpy="${mti10_right_calib_rpy}"/>
 </joint>
 <link name="mti10_imu_link_left"/>
@@ -1063,5 +1063,5 @@
   <parent link="hesai_lidar"/>
   <child link="mti10_imu_link_left"/>
-  <origin xyz="0.295 -0.030 -0.785" rpy="0 1.570796 3.141596"/>
+  <origin xyz="${mti10_left_calib_xyz}" rpy="${mti10_left_calib_rpy}"/>
 </joint>
 <link name="zed_camera_link"/>
@@ -1069,5 +1069,5 @@
   <parent link="hesai_lidar"/>
   <child link="zed_camera_link"/>
-  <origin xyz="0.0 -0.47 -0.1627" rpy="0.0 0.0 -1.57079"/>
+  <origin xyz="${zed2i_calib_xyz}" rpy="${zed2i_calib_rpy}"/>
 </joint>
 <!-- ZED 2i internal frames.
@@ -1157,5 +1157,5 @@
   <parent link="hesai_lidar"/>
   <child link="rsairy"/>
-  <origin xyz="0.125 0.86 0.0" rpy="0.0 -1.91986 -1.5707"/>
+  <origin xyz="${rsairy_calib_xyz}" rpy="${rsairy_calib_rpy}"/>
 </joint>
 <link name="oak"/>
