Commit message: update no collision urdf

File: mtt_description/urdf/robot_no_collision.urdf.xacro (robot description, xacro)
@@ -1,4 +1,6 @@
 <?xml version="1.0"?>
 <robot name="onshape"  xmlns:xacro="https://www.ros.org/wiki/xacro">
+<xacro:arg name="calibration" default="v1"/>
+<xacro:include filename="$(find mtt_description)/urdf/calibrations/calib_$(arg calibration).xacro"/>
     <xacro:macro name="default_transmission" params="joint_name">
         <transmission name="transmission_${joint_name}">
@@ -1021,6 +1023,6 @@
   <origin xyz="-0.7174808381178577409 0.21597831029643155 0.52330103716210749187" rpy="0 0 0"/>
 </joint>
-<!-- Center LiDAR -->
-<link name="center_lidar_link">
+<!-- Hesai XT-32 — direct joint from reference_point (center_lidar_link alias removed) -->
+<link name="hesai_lidar">
   <visual>
     <origin xyz="0 0 0" rpy="0 0 0"/>
@@ -1040,14 +1042,8 @@
   </inertial>
 </link>
-<joint name="center_lidar_joint" type="fixed">
+<joint name="hesai_lidar_joint" type="fixed">
   <parent link="reference_point"/>
-  <child link="center_lidar_link"/>
-  <origin xyz="0.62 -0.266 0.355" rpy="0 0 ${pi/2}"/>
-</joint>
-<link name="hesai_lidar"/>
-<joint name="hesai_lidar_joint" type="fixed">
-  <parent link="center_lidar_link"/>
   <child link="hesai_lidar"/>
-  <origin xyz="0 0 0" rpy="0 0 0"/>
+  <origin xyz="${hesai_calib_xyz}" rpy="${hesai_calib_rpy}"/>
 </joint>
 <link name="imu_link"/>
@@ -1176,7 +1172,7 @@
 </joint>
 <!-- Gazebo sensor plugin for Center LiDAR -->
-<gazebo reference="center_lidar_link">
+<gazebo reference="hesai_lidar">
   <sensor name="center_lidar" type="gpu_lidar">
-    <gz_frame_id>center_lidar_link</gz_frame_id>
+    <gz_frame_id>hesai_lidar</gz_frame_id>
     <pose>0 0 0 0 0 0</pose>
     <update_rate>10</update_rate>
