Commit message: Restore cage orientation and document pending translation check

File: mtt_description/urdf/calibrations/calib_v2.xacro (robot description, xacro)
@@ -2,26 +2,41 @@
 <robot xmlns:xacro="http://www.ros.org/wiki/xacro">
   <!--
-    Calibration v2 — sensor cage AFTER backward displacement.
-    Generated by scripts/calib_hesai_scan.py on 2026-06-26.
+    Calibration v2 — sensor cage after relocation.
+    Position generated by scripts/calib_hesai_scan.py on 2026-06-26.
     xyz = 0.850829 -0.266000 0.355000
     Δ from v1: x=+0.2308 m  y=+0.0000 m  z=+0.0000 m
-    Cage backward shift: -23.1 cm
-    hesai_lidar frame convention (rpy=π): X=BACKWARD, Y=RIGHT, Z=UP.
-    All sensor xyz/rpy below are expressed in this frame.
+    Encoded shift: +23.1 cm along reference_point X (forward in base_link).
+    The original field note described a backward shift. Resolve this discrepancy
+    against the mounting measurement/static bag before accepting the translation.
+    ROTATION FIX (2026-08-27): hesai_calib_rpy was erroneously set to pi (180
+    degrees) here, and imu/mti10/zed2i below were mechanically re-expressed
+    under that wrong assumption (confirmed: each was exactly v1's value
+    rotated 90 degrees about Z, not an independent remeasurement; only rsairy
+    carries a genuine independent post-displacement ICP recalibration). The
+    cage displacement was reported as a pure translation; it never
+    changed hesai_lidar's own rotation. Confirmed live on-robot 2026-08-27:
+    CALIBRATION=v1's rotation (rpy=pi/2) is visually correct in Foxglove
+    (Hesai cloud aligns with camera and URDF); only the position needed the
+    v2 update. hesai_calib_rpy and the cage-internal sensor mounts (imu,
+    mti10, zed2i; unaffected by the cage's own translation) are therefore
+    restored to v1's rotation values. rsairy keeps its independently
+    measured v2 value.
   -->
   <!-- hesai_lidar origin relative to reference_point -->
   <xacro:property name="hesai_calib_xyz" value="0.850829 -0.266000 0.355000"/>
-  <xacro:property name="hesai_calib_rpy" value="0 0 3.141593"/>
-  <!-- IMU (Xsens MTi-100) — in hesai_lidar frame (X=BACKWARD, Y=RIGHT) -->
+  <xacro:property name="hesai_calib_rpy" value="0 0 1.5707963267948966"/>
+  <!-- IMU (Xsens MTi-100) — in hesai_lidar frame (X=LEFT, Y=BACKWARD, matching
+       v1's convention, restored; see ROTATION FIX above) -->
   <xacro:property name="imu_calib_xyz" value="0.0 0.0 0.061"/>
-  <xacro:property name="imu_calib_rpy" value="-3.141593 0 -1.570797"/>
-  <xacro:property name="mti10_right_calib_xyz" value="-0.030 0.295 -0.785"/>
-  <xacro:property name="mti10_right_calib_rpy" value="0 1.570796 -1.570797"/>
-  <xacro:property name="mti10_left_calib_xyz" value="-0.030 -0.295 -0.785"/>
-  <xacro:property name="mti10_left_calib_rpy" value="0 1.570796 1.570797"/>
-  <!-- ZED 2i — in hesai_lidar frame (X=BACKWARD, Y=RIGHT) -->
-  <xacro:property name="zed2i_calib_xyz" value="-0.470 0.0 -0.1627"/>
-  <xacro:property name="zed2i_calib_rpy" value="0 0 -3.141593"/>
-  <!-- RS-Airy — in hesai_lidar frame (X=BACKWARD, Y=RIGHT) -->
+  <xacro:property name="imu_calib_rpy" value="3.141596 0 0"/>
+  <xacro:property name="mti10_right_calib_xyz" value="-0.295 -0.030 -0.785"/>
+  <xacro:property name="mti10_right_calib_rpy" value="0 1.570796 0"/>
+  <xacro:property name="mti10_left_calib_xyz" value="0.295 -0.030 -0.785"/>
+  <xacro:property name="mti10_left_calib_rpy" value="0 1.570796 3.141596"/>
+  <!-- ZED 2i — in hesai_lidar frame (X=LEFT, Y=BACKWARD, restored) -->
+  <xacro:property name="zed2i_calib_xyz" value="0.0 -0.47 -0.1627"/>
+  <xacro:property name="zed2i_calib_rpy" value="0.0 0.0 -1.5707963267948966"/>
+  <!-- RS-Airy — in hesai_lidar frame. KEPT from v2: genuine independent
+       post-displacement recalibration, not derived from a rotation formula. -->
   <!-- Direct ICP v2 (hesai↔rsairy, bag 2026-06-26). P2Pl 4cm voxel. RMSE=3.45cm, Δt=11.6cm. -->
   <!-- z is ill-constrained (no shared vertical structure); x/y/rpy are reliable. -->

File: mtt_description/urdf/robot.urdf.xacro (robot description, xacro)
@@ -1248,6 +1248,6 @@
 <!-- Runtime sensor mounts — all under hesai_lidar so they travel with the cage.
      xyz/rpy values come from calib_*.xacro properties so each calibration version
-     can express positions in its own frame convention (v1: X=LEFT/Y=BACKWARD,
-     v2: X=BACKWARD/Y=RIGHT). -->
+     can express positions in the Hesai frame (X=LEFT/Y=BACKWARD for both
+     v1 and the corrected v2 calibration). -->
 <link name="imu_link"/>
 <joint name="imu_joint" type="fixed">
@@ -1368,5 +1368,5 @@
   <!-- Calibrated 2026-04-21 (P2P→P2Pl→GICP on bag_0.mcap, RMSE=3.07cm at voxel=2cm).
        Values come from calib_*.xacro — expressed in the hesai_lidar frame convention
-       of the active calibration (v1: X=LEFT/Y=BACKWARD, v2: X=BACKWARD/Y=RIGHT). -->
+       of the active calibration (X=LEFT/Y=BACKWARD for v1 and corrected v2). -->
   <origin xyz="${rsairy_calib_xyz}" rpy="${rsairy_calib_rpy}"/>
 </joint>
